File: boards/capture-clip/kicad/capture-clip.kicad_sch (KiCad schematic)
At the start: 52 parts, among them J1 USB-C, J2 LiPo, Q1 AO3401A, SW1 BUTTON, SW2 RESET, U1 ESP32-S3-WROOM-1-N16R8, U2 TP4057, U3 H5VUT2U, U4 RT9080-33GJ5

Commit message: Phase E.3/E.4: capture-clip layout and case, all gates pass; power-path fix (D-025)
30 x 60 mm board routed on the default 8 orders: ERC 0, DRC 0 open, 0 unrouted.
D2 -> RB168MM-40, U4 -> HE9073 (9 V input), C4 10 uF: asleep 12.7 of 20 uA.
Case with battery pocket and a tray-side microphone opening (new pcbgen
[[case.opening]] side = "bottom", board-edge notch); fit.json 30 of 30.
Cost: $66.89 per design for 5 bare + 2 assembled.

Co-Authored-By: Claude Opus 5.5 <noreply@anthropic.com>
Claude-Session: https://claude.ai/code/session_012cDPYugvAySizSnVuzDouS
Parts:
- removed TP9: SPARE_IO21, TestPoint:TestPoint_Pad_D1.5mm, symbol Connector:TestPoint
- added R19: 4.3k, Resistor_SMD:R_0805_2012Metric, symbol Device:R
- C4: value 1u -> 10u; LCSC C28323 -> C15850
- D2: value RB160M-30 -> RB168MM-40; footprint Diode_SMD:D_SOD-123 -> Diode_SMD:D_SOD-123F; LCSC C7502715 -> C509936; MPN RB160M-30 -> RB168MM-40TR
- H1, H2: footprint MountingHole:MountingHole_2.2mm_M2 -> MountingHole:MountingHole_2.5mm
- R6: value 100k -> 10k; LCSC C149504 -> C17414
- TP8: value SPARE_IO7 -> SPARE_IO21
- U4: value RT9080-33GJ5 -> HE9073A33M5R; footprint Package_TO_SOT_SMD:TSOT-23-5 -> Package_TO_SOT_SMD:SOT-23-5; LCSC C841192 -> C723789; MPN RT9080-33GJ5 -> HE9073A33M5R
Connections:
- net CHG_PROG: now also R19.1
- net SPARE_IO21: now also TP8.1
- net SPARE_IO7 renamed CHG_FAST_N
- net CHG_FAST_N: now also R19.2; no longer TP8.1
Other:
- moved on the sheet: C1, C2, D1, R4, R5
