File: boards/starter/kicad/starter.kicad_sch (KiCad schematic)
At the start: 37 parts, among them J1 USB-C, J2 Qwiic, SW1 RESET, SW2 BOOT, U1 ESP32-S3-WROOM-1-N16R8, U2 LDL1117S33R, U3 H5VUT2U, U4 SHT40-AD1B

Commit message: Phase 1 complete: SWIG crash fixed, all gates pass, fab files, reviews
- Segfault root cause: pcbnew's Remove() and Outline()/GetCourtyard() hand
  KiCad-owned memory to Python; fixed (leak removed items, borrowed()).
  Each stage and each SWIG step now runs in its own process; zones are
  filled by kicad-cli (D-011)
- Routing: pours hidden from Freerouting so GND gets real tracks; Power
  class 0.3 mm; retries; stitching checks track clearance (D-012)
- New gates: netlist round trip, net-class patterns, routing report
- fab.py: gerbers/drill zip, JLCPCB BOM and CPL with rotation corrections
- Datasheet check and blind review by separate agents; cap values, fuse
  before TVS, C1 placement, USB net class fixed (D-014)
- Stack survey confirms the stack (D-013)

Co-Authored-By: Claude Opus 5.5 <noreply@anthropic.com>
Claude-Session: https://claude.ai/code/session_01EfFHJzgmcgpgRkWALfogi6
Parts:
- C2: value 22u -> 1u; LCSC C45783 -> C28323
- C3: value 10u -> 22u; LCSC C15850 -> C45783
Connections:
- net +5V: now also D3.1 (A1)
- net VBUS: no longer D3.1 (A1)
Changed lines of the file:
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@@
 	)
 	(symbol
-		(lib_id "power:VBUS")
+		(lib_id "power:+5V")
 		(at 43.18 156.21 180)
 		(unit 1)
@@
 			)
 		)
-		(property "Value" "VBUS"
+		(property "Value" "+5V"
 			(at 43.18 159.41 0)
 			(show_name no)
@@
 			)
 		)
-		(property "Value" "10u"
+		(property "Value" "22u"
 			(at 153.162 124.46 0)
 			(show_name no)
@@
 			)
 		)
-		(property "LCSC" "C15850"
+		(property "LCSC" "C45783"
 			(at 149.86 127 0)
 			(hide yes)
@@
 			)
 		)
-		(property "Value" "22u"
+		(property "Value" "1u"
 			(at 97.282 101.6 0)
 			(show_name no)
@@
 			)
 		)
-		(property "LCSC" "C45783"
+		(property "LCSC" "C28323"
 			(at 93.98 104.14 0)
 			(hide yes)

Commit message: Starter: LDO cooling copper, 0.3 mm ESP32 EPAD holes, 0.75 A fuse (D-015)
- pcbgen: CopperZone (local pour of one net, above GND) and
  RouteOptions.stitch_local (per-net via stitching); routing report now
  lists every pour and vias per net.
- Starter: +3V3 pour on both layers under U2's tab with 20 vias.
- Local footprint lib/footprints/pcbgen.pretty/ESP32-S3-WROOM-1_EPAD-Drill0.3:
  KiCad's footprint with the 12 EPAD drills at 0.3 mm (JLCPCB's quote form
  charges ~$50 for 0.2 mm).
- F1: Bourns MF-NSMF075-2 (C89653), which has a published derating table;
  a 0.5 A PTC holds only ~0.35-0.40 A at 50-60 C.
- Research: research/2026-09-29-holes-and-fuse.md.
- Full run: ERC 0, DRC 0 open (11 waived silk), 0 unrouted.

Co-Authored-By: Claude Opus 5.5 <noreply@anthropic.com>
Claude-Session: https://claude.ai/code/session_01QxXhFJGsvChPbjPevYQU4a
Parts:
- F1: value 500mA -> 750mA; LCSC C720075 -> C89653; MPN JK-nSMD050-30 -> MF-NSMF075-2
- U1: footprint RF_Module:ESP32-S3-WROOM-1 -> pcbgen:ESP32-S3-WROOM-1_EPAD-Drill0.3
Changed lines of the file:
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@@
 			)
 		)
-		(property "Value" "500mA"
+		(property "Value" "750mA"
 			(at 45.72 176.149 0)
 			(show_name no)
@@
 			)
 		)
-		(property "LCSC" "C720075"
+		(property "LCSC" "C89653"
 			(at 45.72 172.72 0)
 			(hide yes)
@@
 			)
 		)
-		(property "MPN" "JK-nSMD050-30"
+		(property "MPN" "MF-NSMF075-2"
 			(at 45.72 172.72 0)
 			(hide yes)
@@
 			)
 		)
-		(property "Footprint" "RF_Module:ESP32-S3-WROOM-1"
+		(property "Footprint" "pcbgen:ESP32-S3-WROOM-1_EPAD-Drill0.3"
 			(at 149.86 68.58 0)
 			(hide yes)

Commit message: Parts search tool and PARTS gate: jlc module, `pcb parts search/show`, MPN + stock check in cost
- crates/pcbgen/src/jlc.rs: JLCPCB parts API client moved out of cost.rs; search with
  Basic / no-fee / in-stock filters and paging (filters verified live), get by exact LCSC
  code, richer Listing (MPN, maker, package, category, description, parameters,
  datasheet + JLCPCB copy, part page), 1-day answer cache in ~/.cache/pcbgen/jlc keyed by
  request-body hash, datasheet download + pdftotext, MPN normaliser.
- New bin `pcb` (cargo run --release -p pcbgen --bin pcb -- parts ...): `parts search`
  table (class with fee, stock, price at qty, package, MPN, KiCad footprint name hint),
  `parts show [--datasheet]`. One module per command under src/bin/pcb/.
- cost stage: PARTS gate (JLCPCB's MPN for each BOM line's LCSC code must match the
  circuit's MPN; stock must cover the order incl. attrition); fails the stage on a
  mismatch, warns on lines without an MPN. `--fresh` skips the cache. cost.json unchanged.
- starter: MPNs from JLCPCB's listings on every assembled part; schematic and board
  regenerated (MPN properties only; routing, BOM, CPL and gerber copper identical).

Co-Authored-By: Claude Opus 5.5 <noreply@anthropic.com>
Claude-Session: https://claude.ai/code/session_01T5c1vQNCB4AARjsQRobsDT
Parts:
- C1: MPN (none) -> CL21A106KAYNNNE
- C2, C5: MPN (none) -> CL21B105KBFNNNE
- C3: MPN (none) -> CL21A226MAQNNNE
- C4, C6: MPN (none) -> CC0805KRX7R9BB104
- D1: MPN (none) -> KT-0805G
- D2: MPN (none) -> NCD0805R1
- R1, R2: MPN (none) -> 0805W8F5101T5E
- R3, R6: MPN (none) -> 0805W8F1001T5E
- R4, R5: MPN (none) -> 0805W8F1002T5E
- R7, R8: MPN (none) -> 0805W8F4701T5E
- SW1, SW2: MPN (none) -> TS-1187A-B-A-B
Changed lines of the file:
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@@
 	(title_block
 		(title "ESP32-S3 starter board")
-		(date "2026-09-29")
+		(date "2026-10-01")
 		(rev "0")
 		(comment 1 "Generated from code by pcbgen; do not edit by hand")
@@
 			)
 		)
+		(property "MPN" "CC0805KRX7R9BB104"
+			(at 287.02 86.36 0)
+			(hide yes)
+			(show_name no)
+			(do_not_autoplace no)
+			(effects
+				(font
+					(size 1.27 1.27)
+				)
+			)
+		)
 		(pin "1"
 		)
@@
 			)
 		)
+		(property "MPN" "KT-0805G"
+			(at 91.44 139.7 0)
+			(hide yes)
+			(show_name no)
+			(do_not_autoplace no)
+			(effects
+				(font
+					(size 1.27 1.27)
+				)
+			)
+		)
 		(pin "1"
 		)
@@
 			)
 		)
+		(property "MPN" "CL21A226MAQNNNE"
+			(at 149.86 127 0)
+			(hide yes)
+			(show_name no)
+			(do_not_autoplace no)
+			(effects
+				(font
+					(size 1.27 1.27)
+				)
+			)
+		)
 		(pin "1"
 		)
@@
 			)
 		)
+		(property "MPN" "0805W8F4701T5E"
+			(at 284.48 121.92 0)
+			(hide yes)
+			(show_name no)
+			(do_not_autoplace no)
+			(effects
+				(font
+					(size 1.27 1.27)
+				)
+			)
+		)
 		(pin "1"
 		)
@@
 			)
 		)
+		(property "MPN" "CL21B105KBFNNNE"
+			(at 149.86 203.2 0)
+			(hide yes)
+			(show_name no)
+			(do_not_autoplace no)
+			(effects
+				(font
+					(size 1.27 1.27)
+				)
+			)
+		)
 		(pin "1"
 		)
@@
 			)
 		)
+		(property "MPN" "TS-1187A-B-A-B"
+			(at 200.66 35.56 0)
+			(hide yes)
+			(show_name no)
+			(do_not_autoplace no)
+			(effects
+				(font
+					(size 1.27 1.27)
+				)
+			)
+		)
 		(pin "1"
 		)
@@
 			)
 		)
+		(property "MPN" "TS-1187A-B-A-B"
+			(at 200.66 63.5 0)
+			(hide yes)
+			(show_name no)
+			(do_not_autoplace no)
+			(effects
+				(font
+					(size 1.27 1.27)
+				)
+			)
+		)
 		(pin "1"
 		)
@@
 			)
 		)
+		(property "MPN" "0805W8F1002T5E"
+			(at 200.66 48.26 0)
+			(hide yes)
+			(show_name no)
+			(do_not_autoplace no)
+			(effects
+				(font
+					(size 1.27 1.27)
+				)
+			)
+		)
 		(pin "1"
 		)
@@
 			)
 		)
+		(property "MPN" "CL21A106KAYNNNE"
+			(at 93.98 71.12 0)
+			(hide yes)
+			(show_name no)
+			(do_not_autoplace no)
+			(effects
+				(font
+					(size 1.27 1.27)
+				)
+			)
+		)
 		(pin "1"
 		)
@@
 			)
 		)
+		(property "MPN" "0805W8F1001T5E"
+			(at 91.44 124.46 0)
+			(hide yes)
+			(show_name no)
+			(do_not_autoplace no)
+			(effects
+				(font
+					(size 1.27 1.27)
+				)
+			)
+		)
 		(pin "1"
 		)
@@
 			)
 		)
+		(property "MPN" "CC0805KRX7R9BB104"
+			(at 149.86 157.48 0)
+			(hide yes)
+			(show_name no)
+			(do_not_autoplace no)
+			(effects
+				(font
+					(size 1.27 1.27)
+				)
+			)
+		)
 		(pin "1"
 		)
@@
 			)
 		)
+		(property "MPN" "0805W8F1002T5E"
+			(at 149.86 180.34 0)
+			(hide yes)
+			(show_name no)
+			(do_not_autoplace no)
+			(effects
+				(font
+					(size 1.27 1.27)
+				)
+			)
+		)
 		(pin "1"
 		)
@@
 			)
 		)
+		(property "MPN" "0805W8F1001T5E"
+			(at 241.3 35.56 0)
+			(hide yes)
+			(show_name no)
+			(do_not_autoplace no)
+			(effects
+				(font
+					(size 1.27 1.27)
+				)
+			)
+		)
 		(pin "1"
 		)
@@
 			)
 		)
+		(property "MPN" "CL21B105KBFNNNE"
+			(at 93.98 104.14 0)
+			(hide yes)
+			(show_name no)
+			(do_not_autoplace no)
+			(effects
+				(font
+					(size 1.27 1.27)
+				)
+			)
+		)
 		(pin "1"
 		)
@@
 			)
 		)
+		(property "MPN" "0805W8F5101T5E"
+			(at 43.18 104.14 0)
+			(hide yes)
+			(show_name no)
+			(do_not_autoplace no)
+			(effects
+				(font
+					(size 1.27 1.27)
+				)
+			)
+		)
 		(pin "1"
 		)
@@
 			)
 		)
+		(property "MPN" "0805W8F4701T5E"
+			(at 284.48 106.68 0)
+			(hide yes)
+			(show_name no)
+			(do_not_autoplace no)
+			(effects
+				(font
+					(size 1.27 1.27)
+				)
+			)
+		)
 		(pin "1"
 		)
@@
 			)
 		)
+		(property "MPN" "0805W8F5101T5E"
+			(at 43.18 91.44 0)
+			(hide yes)
+			(show_name no)
+			(do_not_autoplace no)
+			(effects
+				(font
+					(size 1.27 1.27)
+				)
+			)
+		)
 		(pin "1"
 		)
@@
 			(at 238.76 48.26 0)
 			(hide yes)
+			(show_name no)
+			(do_not_autoplace no)
+			(effects
+				(font
+					(size 1.27 1.27)
+				)
+			)
+		)
+		(property "MPN" "NCD0805R1"
+			(at 238.76 48.26 0)
+			(hide yes)
